File: kicad/circuits/circuits.kicad_sch (KiCad schematic)
At the start: 177 parts

Commit message: Updated schematic
Parts:
- removed C? (x10): C, symbol Device:C
- removed R? (x35): R_Trim, symbol Device:R_Trim
- removed R?: (no value), symbol Device:R_Trim
- removed R?: R, symbol Device:R
- added C? (x10): 100n, symbol Device:C
- added J?: (no value), symbol Connector:USB_C_Receptacle
- added R? (x15): (no value), symbol Device:R
- added R? (x3): R, symbol Device:R
- added R? (x2): 1k87, symbol Device:R
- added R? (x2): 768, symbol Device:R
- added R? (x2): 576, symbol Device:R
- added R? (x2): 931, symbol Device:R
- added R? (x2): 1k82, symbol Device:R
- added R? (x2): 3k65, symbol Device:R
- added R? (x2): 73.2, symbol Device:R
- added R? (x2): 137, symbol Device:R
- added R? (x2): 1k54, symbol Device:R
- added RV?: R_Potentiometer, symbol Device:R_Potentiometer
- added RV?: (no value), symbol Device:R_Potentiometer
- added U? (x2): LM358, symbol Amplifier_Operational:LM358
- C?: value (none) -> C
- C? (x12): value C -> (none)
- D?: value (none) -> LED
- R? (x5): value (none) -> 100k
- R? (x2): value (none) -> R
- RV? (x2): value (none) -> 2k2
- U? (x2): value (none) -> LM339
Connections:
- net +5V: now also J?.A4 (VBUS), J?.A9 (VBUS), J?.B4 (VBUS), J?.B9 (VBUS)
- net GND: now also C?.2, C?.2, C?.2, C?.2, C?.2, J?.A1 (GND), J?.A12 (GND), J?.B1 (GND), J?.B12 (GND), J?.S1 (SHIELD), R?.2, R?.2, R?.2, R?.2, R?.2, R?.2, R?.2, R?.2, R?.2, U?.3 (+), U?.3 (+)
- net at C?.1, C?.2: now also R?.1 (x3)
- net at U?.1, U?.2 (-): now also R?.1, R?.2 (x6)
- net at C?.2, U?.3 (+): now also R?.1 (x4)
- net at U?.1, U?.2 (-), U?.5 (+)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: now also R?.2 (x4)
- net at C?.1, C?.1: now also R?.1, R?.2 (x4)
- net at C?.1, RV?.2, U?.1: now also R?.1, R?.1, R?.1, R?.1
- net at C?.1: now also R?.1, R?.2 (x3)
- net at C?.2, U?.3 (+): now also R?.2 (x3)
- net at C?.1, U?.1, U?.2 (-): now also R?.2 (x2)
- net at U?.3 (+): now also C?.2, R?.1 (x5)
- net at C?.2, U?.1, U?.2 (-): now also R?.1 (x2)
- net audio_in renamed audio_in_L
- net audio_in_L: now also RV?.3, RV?.3
- new net: C?.1, C?.1, R?.1, R?.2 (x5)
- new net: RV?.1, U?.1 (x2)
- new net: RV?.2, U?.2 (-) (x2)

Commit message: Added some new values to schematic
Parts:
- added C1, C12, C13, C14, C19, C2, C20, C21, C22, C25, C26, C28, C3, C32, C33, C34, C39, C4, C40, C41, C42, C45, C46, C48, C5, C52, C53, C54, C59, C6, C60, C61, C62, C65, C66, C8: (no value), symbol Device:C
- added D10, D16, D17, D18, D19, D20, D26, D27, D28, D29, D30, D36, D37, D38, D39, D40, D6, D7, D8, D9: (no value), symbol Device:LED
- added J2, J3: (no value), symbol Connector:AudioJack3
- added J4, J5: (no value), symbol Connector:Screw_Terminal_01x02
- added R1, R10, R103, R104, R105, R106, R107, R108, R109, R11, R110, R111, R112, R12, R123, R124, R125, R126, R127, R128, R129, R130, R131, R132, R14, R143, R144, R145, R146, R147, R148, R149, R150, R151, R152, R163, R164, R165, R166, R167, R168, R169, R170, R171, R172, R2, R23, R24, R25, R26, R27, R28, R29, R3, R30, R35, R36, R37, R38, R4, R40, R49, R50, R51, R52, R53, R54, R55, R56, R61, R62, R63, R64, R66, R75, R76, R77, R78, R79, R80, R81, R82, R88, R89, R9, R90, R91, R92: (no value), symbol Device:R
- added RV14, RV15, RV16, RV17, RV18, RV3, RV4, RV8: (no value), symbol Device:R_Potentiometer
- added RV5, RV6: (no value), symbol Device:R_Potentiometer_Dual_Separate
- added U10, U16, U17, U18, U19, U20, U26, U27, U28, U29, U3, U30, U36, U37, U38, U39, U4, U40, U5, U6, U7, U8: (no value), symbol Amplifier_Operational:LM358
- added U46, U47, U48, U49, U50, U56, U57, U58, U59, U60: (no value), symbol Comparator:LM339
- C15, C27, C35, C47, C55, C7: renamed from C?; value C -> (none)
- C16, C29, C30, C36, C37, C49, C50, C56, C57, C9: renamed from C?; value 100n -> (none)
- D1, D11, D12, D13, D14, D15, D2, D21, D22, D23, D24, D25, D3, D31, D32, D33, D34, D35, D4, D5: renamed from D?; value LED -> (none)
- R100, R102, R113, R114, R115, R116, R117, R133, R134, R135, R136, R137, R15, R158, R159, R16, R160, R161, R162, R41, R42, R67, R68, R94, R96, R98: renamed from R?; value R -> (none)
- R101, R118, R119, R120, R121, R122, R138, R139, R140, R141, R142, R153, R154, R155, R156, R157, R83, R84, R85, R86, R87, R93, R95, R97, R99: renamed from R?; value 100k -> (none)
- R31, R57: renamed from R?; value 931 -> (none)
- R32, R58: renamed from R?; value 1k82 -> (none)
- R33, R59: renamed from R?; value 768 -> (none)
- R43, R69: renamed from R?; value 137 -> (none)
- R44, R70: renamed from R?; value 1k87 -> (none)
- R45, R71: renamed from R?; value 576 -> (none)
- R46, R72: renamed from R?; value 3k65 -> (none)
- R47, R73: renamed from R?; value 73.2 -> (none)
- R48, R74: renamed from R?; value 1k54 -> (none)
- RV10, RV11, RV12, RV13, RV7, RV9: renamed from RV?; value 2k2 -> (none)
- RV2: renamed from RV?; value R_Potentiometer -> (none)
- U1, U11, U12, U13, U14, U15, U2, U21, U22, U23, U24, U25, U31, U32, U33, U34, U35, U9: renamed from U?; value LM358 -> (none)
- U41, U42, U43, U44, U45, U51, U52, U53, U54, U55: renamed from U?; value LM339 -> (none)
- gave numbers to parts that had none: 31
Connections:
- net +12V: now also RV14.1, RV15.1, RV16.1, RV17.1, RV18.1
- net +5V: now also R104.1, R106.1, R108.1, R110.1, R112.1, R123.2, R124.2, R125.2, R126.2, R127.2, R143.2, R144.2, R145.2, R146.2, R147.2, R168.2, R169.2, R170.2, R171.2, R172.2
- net GND: now also C12.2, C13.2, C14.2, C26.1, C32.2, C33.2, C34.2, C46.1, C52.2, C53.2, C54.2, C66.1, J2.S, J3.S, J4.2 (Pin_2), J5.2 (Pin_2), R163.2, R164.2, R165.2, R166.2, R167.2, R24.2, R26.2, R28.2, R30.2, R50.2, R52.2, R54.2, R56.2, R76.2, R78.2, R80.2, R82.2, RV14.3, RV15.3, RV16.3, RV17.3, RV18.3, RV5.3, RV6.3, RV8.3, U3.3 (+), U4.3 (+)
- net audio_in_L: now also C1.1, C3.1, C5.1; no longer RV1.3, RV2.3
- net at RV2.1, U2.1: now also J2.R
- net at RV1.1, U1.1: now also J2.T
- new net: J4.1 (Pin_1), R1.2, R3.1, RV5.1
- new net: C8.1, R10.1, R11.1, R12.1, R9.1, RV8.2, U10.1
- new net: C19.1, C8.2, R23.1
- new net: R131.2, R151.1, U59.4 (-)
- new net: R151.2, R166.1, U59.6 (-)
- new net: C12.1, C20.1, R25.1, R9.2
- new net: C20.2, R26.1, U17.3 (+)
- new net: C62.2, R82.1, U39.3 (+)
- new net: C48.2, C59.1, R75.1
- new net: R75.2, U36.1, U36.2 (-), U46.5 (+), U46.7 (+), U56.5 (+), U56.7 (+)
- new net: C14.1, C22.1, R11.2, R29.1
- new net: C22.2, R30.1, U19.3 (+)
- new net: C65.2, U40.1, U40.2 (-), U50.5 (+), U50.7 (+), U60.5 (+), U60.7 (+)
- new net: C66.2, R66.2, U40.3 (+)
- new net: D19.1 (K), U49.1
- new net: D19.2 (A), R126.1
- new net: R51.2, R61.1, U27.1, U27.2 (-)
- new net: C52.1, C60.1, R61.2, R77.1
- new net: C48.1, R49.2, U26.1, U26.2 (-)
- new net: C39.2, R50.1, U26.3 (+)
- new net: R29.2, R37.1, U19.1, U19.2 (-)
- new net: C34.1, C42.1, R37.2, R55.1
- new net: C59.2, R76.1, U36.3 (+)
- new net: R25.2, R35.1, U17.1, U17.2 (-)
- new net: R88.1, RV14.2
- new net: R103.1, R88.2, U46.4 (-)
- new net: R105.2, R129.1, U47.6 (-)
- new net: R129.2, R149.1, U57.4 (-)
- new net: R53.2, R62.1, U28.1, U28.2 (-)
- new net: C53.1, C61.1, R62.2, R79.1
- new net: R1.1, U5.1, U7.3 (+)
- new net: RV5.2, U5.2 (-)
- new net: C5.2, U5.3 (+)
- new net: C25.1, R12.2, R14.1
- new net: C65.1, R64.2, R66.1
- new net: C33.1, C41.1, R36.2, R53.1
- new net: C41.2, R54.1, U28.3 (+)
- new net: C54.1, C62.1, R63.2, R81.1
- new net: C28.2, C39.1, R49.1
- new net: C40.2, R52.1, U27.3 (+)
- new net: RV8.1, U10.2 (-)
- new net: R105.1, R89.2, U47.4 (-)
- new net: J3.R, RV4.1, U4.1
- new net: RV4.2, U4.2 (-)
- new net: R2.1, U6.1, U8.3 (+)
- new net: J5.1 (Pin_1), R2.2, R4.1, RV6.1
- new net: C45.1, R38.2, R40.1
- new net: C46.2, R40.2, U30.3 (+)
- new net: R77.2, U37.1, U37.2 (-), U47.5 (+), U47.7 (+), U57.5 (+), U57.7 (+)
- new net: D16.1 (K), U46.1
- new net: D16.2 (A), R123.1
- new net: D40.1 (K), U60.1
- new net: D40.2 (A), R172.1
- new net: R91.1, RV17.2
- new net: D26.1 (K), U56.2
- new net: R128.2, R148.1, U56.4 (-)
- new net: R92.1, RV18.2
- new net: C2.2, RV2.3
- new net: C28.1, R23.2, U16.1, U16.2 (-)
- new net: C13.1, C21.1, R10.2, R27.1
- new net: D39.1 (K), U59.1
- new net: D39.2 (A), R171.1
- new net: D8.1 (K), U48.2
- new net: D8.2 (A), R108.2
- new net: D9.1 (K), U49.2
- new net: D9.2 (A), R110.2
- new net: R111.1, R92.2, U50.4 (-)
- new net: R111.2, R132.1, U50.6 (-)
- new net: D17.2 (A), R124.1
- new net: C42.2, R56.1, U29.3 (+)
- new net: D37.2 (A), R169.1
- new net: D18.2 (A), R125.1
- new net: C45.2, R64.1, U30.1, U30.2 (-)
- new net: J3.T, RV3.1, U3.1
- new net: R109.2, R131.1, U49.6 (-)
- new net: D29.1 (K), U59.2
- new net: R81.2, U39.1, U39.2 (-), U49.5 (+), U49.7 (+), U59.5 (+), U59.7 (+)
- new net: R132.2, R152.1, U60.4 (-)
- new net: D37.1 (K), U57.1
- new net: R79.2, U38.1, U38.2 (-), U48.5 (+), U48.7 (+), U58.5 (+), U58.7 (+)
- new net: C61.2, R80.1, U38.3 (+)
- new net: C60.2, R78.1, U37.3 (+)
- new net: C21.2, R28.1, U18.3 (+)
- new net: R109.1, R91.2, U49.4 (-)
- new net: R55.2, R63.1, U29.1, U29.2 (-)
- new net: R89.1, RV15.2
- new net: D26.2 (A), R143.1
- new net: D20.1 (K), U50.1
- new net: D20.2 (A), R127.1
- new net: R148.2, R163.1, U56.6 (-)
- new net: R107.2, R130.1, U48.6 (-)
- new net: R130.2, R150.1, U58.4 (-)
- new net: C25.2, R38.1, U20.1, U20.2 (-)
- new net: D29.2 (A), R146.1
- new net: D27.1 (K), U57.2
- new net: D27.2 (A), R144.1
- new net: D36.1 (K), U56.1
- new net: D36.2 (A), R168.1
- new net: R152.2, R167.1, U60.6 (-)
- new net: D10.2 (A), R112.2
- new net: D6.1 (K), U46.2
- new net: D6.2 (A), R104.2
- new net: R90.1, RV16.2
- new net: C26.2, R14.2, U20.3 (+)
- new net: D10.1 (K), U50.2
- new net: D38.1 (K), U58.1
- new net: R150.2, R165.1, U58.6 (-)
- new net: D38.2 (A), R170.1
- new net: C4.2, RV4.3
- new net: R149.2, R164.1, U57.6 (-)
- new net: R107.1, R90.2, U48.4 (-)
- new net: R103.2, R128.1, U46.6 (-)
- new net: D28.1 (K), U58.2
- new net: R4.2, U8.1, U8.2 (-)
- new net: RV6.2, U6.2 (-)
- new net: R3.2, U7.1, U7.2 (-)
- new net: D30.1 (K), U60.2
- new net: C32.1, C40.1, R35.2, R51.1
- new net: C1.2, RV1.3
- new net: R27.2, R36.1, U18.1, U18.2 (-)
- new net: RV3.2, U3.2 (-)
- new net: C3.2, RV3.3
- new net: D18.1 (K), U48.1
- new net: D17.1 (K), U47.1
- new net: D7.1 (K), U47.2
- new net: D7.2 (A), R106.2
- new net: D30.2 (A), R147.1
- new net: D28.2 (A), R145.1
- new net: C6.2, U6.3 (+)
- new net: C19.2, R24.1, U16.3 (+)
- new net audio_in_R: C2.1, C4.1, C6.1, U10.3 (+)
Other:
- note added: "Headphone Amp 1"
- note added: "Headphone Amp 2"
- note added: "Probably should be done more properly. Too bard. Just don't plug it into a low power port"
- note added: "Speaker Amp"
- note added: "https://e2e.ti.com/blogs_/archives/b/thesignal/posts/paralleling-op-amps-is-it-possible"
