File: kicad/band-pass-high/band-pass-high.kicad_sch (KiCad schematic)
At the start: 66 parts, among them J1 Conn_01x06

Commit message: Made a filter PCB design
Parts:
- removed D1, D5: blue, symbol Device:LED
- removed D2, D6: green, symbol Device:LED
- removed D3, D7: yellow, symbol Device:LED
- removed D4, D8: orange, symbol Device:LED
- removed R19, R20, R21, R22, R23: 100k, symbol Device:R
- removed R24, R25, R26, R27, R7, R8, R9: R, symbol Device:R
- removed R6: BLUe, symbol Device:R
- removed RV2: (no value), symbol Device:R_Potentiometer
- added J?: Conn_01x09_Male, Connector_PinHeader_2.54mm:PinHeader_1x09_P2.54mm_Horizontal, symbol Connector:Conn_01x09_Male
- J1: footprint (none) -> Connector_PinHeader_2.54mm:PinHeader_1x06_P2.54mm_Horizontal
- R1, R10, R11, R12, R13, R14, R15, R16, R17, R18, R2, R28, R29, R3, R30, R31, R32, R33, R34, R35, R36, R4, R5: footprint (none) -> Resistor_SMD:R_1206_3216Metric
- RV1: value (none) -> 10k; footprint (none) -> Potentiometer_THT:Potentiometer_Runtron_RM-065_Vertical
- U1, U2, U3: value (none) -> LF353DR; footprint (none) -> Package_SO:SOIC-8_3.9x4.9mm_P1.27mm
- U4, U5: value (none) -> LM339DR; footprint (none) -> Package_SO:SO-14_3.9x8.65mm_P1.27mm
Connections:
- net +5V: now also J?.5 (Pin_5)
- net at U5.7 (+): now also R2.2, R3.1, U4.7 (+)
- net at U5.11 (+): now also R3.2, R4.1, U4.11 (+)
- net at U5.5 (+): now also R1.2, R2.1, U4.5 (+)
- net at U4.1: now also J?.2 (Pin_2)
- net at U5.14: now also J?.9 (Pin_9)
- net at U4.2: now also J?.1 (Pin_1)
- net at U5.13: now also J?.8 (Pin_8)
- net at U5.9 (+): now also R4.2, R5.1, U4.9 (+)
- net at U4.14: now also J?.4 (Pin_4)
- net at U5.1: now also J?.7 (Pin_7)
- net at U5.2: now also J?.6 (Pin_6)
- net at U4.13: now also J?.3 (Pin_3)
Other:
- note added: "High"
- note added: "Low"

Commit message: Updated something I think ...
Parts:
- gave numbers to parts that had none: 1
Changed lines of the file:
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@@
   (symbol (lib_id "Connector:Conn_01x09_Male") (at 698.5 370.84 0) (mirror y) (unit 1)
     (in_bom yes) (on_board yes) (fields_autoplaced)
-    (property "Reference" "J?" (id 0) (at 699.2112 368.7369 0)
+    (property "Reference" "J2" (id 0) (at 699.2112 368.7369 0)
       (effects (font (size 1.27 1.27)) (justify right))
     )
@@
     )
     (path "/c1386bdf-4187-47e0-8dd8-3dad8c4589c6"
-      (reference "J?") (unit 1) (value "Conn_01x09_Male") (footprint "Connector_PinHeader_2.54mm:PinHeader_1x09_P2.54mm_Horizontal")
+      (reference "J2") (unit 1) (value "Conn_01x09_Male") (footprint "Connector_PinHeader_2.54mm:PinHeader_1x09_P2.54mm_Horizontal")
     )
     (path "/b730191b-a000-46b2-82d0-fb5a460f105a"
