File: kicad/power/power.kicad_sch (KiCad schematic)
At the start: 45 parts, among them J1 Conn_01x06, J2 Conn_01x09_Male, U1 LF353DR, U2 LF353DR, U3 LF353DR, U4 LM339DR, U5 LM339DR

Commit message: Updated some power stuff
Parts:
- removed C1, C10, C11, C12, C2, C3, C4, C5, C6, C7, C8, C9: 100n, Capacitor_SMD:C_1206_3216Metric, symbol Device:C
- removed J2: Conn_01x09_Male, Connector_PinHeader_2.54mm:PinHeader_1x09_P2.54mm_Horizontal, symbol Connector:Conn_01x09_Male
- removed R1, R2, R3, R4, R5: 100k, Resistor_SMD:R_1206_3216Metric, symbol Device:R
- removed R10, R11, R12, R28, R29, R30: 137, Resistor_SMD:R_1206_3216Metric, symbol Device:R
- removed R13, R14, R15, R31, R32, R33: 931, Resistor_SMD:R_1206_3216Metric, symbol Device:R
- removed R16, R17, R18, R34, R35, R36: 1k87, Resistor_SMD:R_1206_3216Metric, symbol Device:R
- removed RV1, RV3, RV4: 10k, Potentiometer_THT:Potentiometer_Runtron_RM-065_Vertical, symbol Device:R_Potentiometer
- removed U1, U2, U3: LF353DR, Package_SO:SOIC-8_3.9x4.9mm_P1.27mm, symbol Amplifier_Operational:LM358
- removed U4, U5: LM339DR, Package_SO:SO-14_3.9x8.65mm_P1.27mm, symbol Comparator:LM339
- added C? (x2): C, symbol Device:C
- added J?: Conn_01x02_Male, symbol Connector:Conn_01x02_Male
- added J? (x2): Screw_Terminal_01x02, symbol Connector:Screw_Terminal_01x02
- added J? (x3): AudioJack3, symbol Connector:AudioJack3
- added J?: USB_C_Receptacle, symbol Connector:USB_C_Receptacle
- added J?: Conn_01x03_Male, symbol Connector:Conn_01x03_Male
- added R? (x4): 20, symbol Device:R
- added RV? (x4): R_Potentiometer, symbol Device:R_Potentiometer
- added RV? (x2): 2k2, symbol Device:R_Potentiometer
- added RV? (x2): R_Potentiometer_Dual_Separate, symbol Device:R_Potentiometer_Dual_Separate
- added U? (x2): LF353DR, symbol Amplifier_Operational:LM358
- added U? (x8): LM4565F-GE2, symbol Amplifier_Operational:LM358
Connections:
- net +15V: now also J?.1 (Pin_1)
- net +5V: now also J?.2 (Pin_2), J?.A4 (VBUS), J?.A9 (VBUS), J?.B4 (VBUS), J?.B9 (VBUS)
- net -15V: now also J?.3 (Pin_3)
- net GND: now also J?.1 (Pin_1), J?.2 (Pin_2), J?.2 (Pin_2), J?.2 (Pin_2), J?.A1 (GND), J?.A12 (GND), J?.B1 (GND), J?.B12 (GND), J?.S, J?.S, J?.S, J?.S1 (SHIELD), RV?.3, RV?.3, RV?.3, RV?.3, U?.3 (+), U?.3 (+), U?.3 (+), U?.3 (+)
- net audio_left: now also J1.2 (Pin_2)
- net audio_right: now also J1.1 (Pin_1)
- new net: J?.T, RV?.1, U?.1 (x2)
- new net: RV?.2, U?.2 (-) (x6)
- new net: RV?.2, U?.1 (x2)
- new net: RV?.1, U?.2 (-) (x2)
- new net: C?.1, J?.R
- new net: J?.1 (Pin_1), R?.1, R?.2, RV?.1 (x2)
- new net: J?.R, RV?.1, U?.1 (x2)
- new net: R?.2, U?.1, U?.2 (-) (x2)
- new net: C?.1, J?.T
- new net: R?.1, U?.1, U?.3 (+) (x2)
- new net audio_in_L: C?.2, RV?.3, RV?.3, U?.3 (+), U?.3 (+)
- new net audio_in_R: C?.2, RV?.3, RV?.3, U?.3 (+), U?.3 (+)
Other:
- note added: "Boost Converter"
- note added: "Headphone Amp 1"
- note added: "Headphone Amp 2"
- note added: "Probably should be done more properly. Too bard. Just don't plug it into a low power port"
- note added: "Speaker Amp"
- note added: "https://e2e.ti.com/blogs_/archives/b/thesignal/posts/paralleling-op-amps-is-it-possible"
- note removed: "1700 - 5000"
- note removed: "High"
- note removed: "Low"
- moved on the sheet: J1
