File: kicad/power/power.kicad_sch (KiCad schematic)
At the start: 32 parts, among them J1 Conn_01x06, J10 Conn_01x06, J11 Conn_01x06, J12 Conn_01x06, J13 Conn_01x06, J2 AudioJack3, J3 USB_C_Receptacle, J4 AudioJack3, J5 AudioJack3, J6 Conn_01x05_Male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

Commit message: Power schematic to pcb update
Parts:
- removed J8: Screw_Terminal_01x02, symbol Connector:Screw_Terminal_01x02
- J1, J10, J11, J12, J13: footprint Connector_PinHeader_2.54mm:PinHeader_1x06_P2.54mm_Horizontal -> Connector_PinHeader_2.54mm:PinHeader_1x06_P2.54mm_Vertical
- J3: footprint (none) -> audio_footprint:usb_footprint
- J6: footprint (none) -> Connector_PinHeader_2.54mm:PinHeader_1x05_P2.54mm_Vertical
- J7: footprint (none) -> TerminalBlock:TerminalBlock_bornier-4_P5.08mm; symbol Connector:Screw_Terminal_01x02 -> Connector:Screw_Terminal_01x04
- J9: value Conn_01x03_Male -> Conn_01x04_Male; footprint (none) -> Connector_PinHeader_2.54mm:PinHeader_1x04_P2.54mm_Vertical
Connections:
- net GND: now also J7.3 (Pin_3)
- net speaker_left: now reaches J7.1 (Pin_1), R1.2, R3.1, RV5.1
- net speaker_right: now reaches R2.2, R4.1, RV6.1
- net speaker_right: now also J7.4 (Pin_4)

Commit message: Made some new stuffs
Parts:
- removed J5: AudioJack3, audio_footprint:audio_jack, symbol Connector:AudioJack3
- removed J7: Screw_Terminal_01x02, TerminalBlock:TerminalBlock_bornier-4_P5.08mm, symbol Connector:Screw_Terminal_01x04
- removed R3, R4: 20, Resistor_SMD:R_1206_3216Metric, symbol Device:R
- removed RV1, RV2, RV3, RV4, RV5, RV6: R_Potentiometer, Potentiometer_THT:Potentiometer_Runtron_RM-065_Vertical, symbol Device:R_Potentiometer
- removed RV7, RV8: 2k2, Potentiometer_THT:Potentiometer_Runtron_RM-065_Vertical, symbol Device:R_Potentiometer
- removed U2, U3, U4: LM4565F-GE2, Package_SO:SOP-8_3.9x4.9mm_P1.27mm, symbol Amplifier_Operational:LM358
- added RV1, RV2: R_Potentiometer_Dual_Separate, Potentiometer_THT:Potentiometer_Alpha_RD902F-40-00D_Dual_Vertical, symbol Device:R_Potentiometer_Dual_Separate
- C1, C2: value C -> 1u
- R1, R2: value 20 -> 100k
Connections:
- net speaker_left is gone; now on net GND: R1.2
- net speaker_right is gone; now on net GND: R2.2
- net +15V: now also J9.4 (Pin_4); no longer J9.1 (Pin_1)
- net -15V: now also J9.1 (Pin_1); no longer J9.4 (Pin_4)
- net GND: now also RV1.3, RV1.6, RV2.3, RV2.6; no longer U1.3 (+), U1.5 (+)
- net audio_in_L: now also R1.1, U1.3 (+)
- net audio_in_R: now also R2.1, U1.5 (+)
- net audio_lefT: now also RV2.2
- net audio_right: now also RV2.5
- net at J4.T, U1.1: now also RV1.2
- net at U1.2 (-): now also RV1.1
- net at U5.6 (-): now also RV2.4
- net at U5.2 (-): now also RV2.1
- net at U1.6 (-): now also RV1.4
- net at J4.R, U1.7: now also RV1.5
- net -5V: no longer names the net of J6.1 (Pin_1)
- no-connect marks 0 -> 1
Other:
- note removed: "Headphone Amp 2"
- note removed: "Speaker Amp"
- note removed: "https://e2e.ti.com/blogs_/archives/b/thesignal/posts/paralleling-op-amps-is-it-possible"
- moved on the sheet: C2, U5C

Commit message: Made new power board
Parts:
- added C4, C6: C, Capacitor_SMD:C_1206_3216Metric, symbol Device:C
- added J5: Conn_01x02_Male, Connector_PinHeader_2.54mm:PinHeader_1x02_P2.54mm_Vertical, symbol Connector:Conn_01x02_Male
- added RV3: R_Potentiometer, Potentiometer_THT:Potentiometer_Runtron_RM-065_Vertical, symbol Device:R_Potentiometer
- added U2: LM7812_TO220, Package_TO_SOT_THT:TO-220-3_Vertical, symbol Regulator_Linear:LM7812_TO220
- added U3: LM337_TO220, Package_TO_SOT_THT:TO-220-3_Vertical, symbol Regulator_Linear:LM337_TO220
- RV1, RV2: footprint Potentiometer_THT:Potentiometer_Alpha_RD902F-40-00D_Dual_Vertical -> audio_footprint:volume-pot
Connections:
- net +15V: now also U2.1 (VI); no longer J1.4 (Pin_4), J10.4 (Pin_4), J11.4 (Pin_4), J12.4 (Pin_4), J13.4 (Pin_4), U1.8 (V+), U5.8 (V+)
- net +5V: now also J5.1 (Pin_1); no longer J3.A4 (VBUS), J3.A9 (VBUS), J3.B4 (VBUS), J3.B9 (VBUS)
- net -15V: now also U3.2 (VI); no longer J1.6 (Pin_6), J10.6 (Pin_6), J11.6 (Pin_6), J12.6 (Pin_6), J13.6 (Pin_6), U1.4 (V-), U5.4 (V-)
- net GND: now also C4.1, C6.2, RV3.3, U2.2 (GND)
- new net: J3.A4 (VBUS), J3.A9 (VBUS), J3.B4 (VBUS), J3.B9 (VBUS), J5.2 (Pin_2)
- new net: RV3.2, U3.1 (ADJ)
- new net +12V: C6.1, J1.4 (Pin_4), J10.4 (Pin_4), J11.4 (Pin_4), J12.4 (Pin_4), J13.4 (Pin_4), U1.8 (V+), U2.3 (VO), U5.8 (V+)
- new net -12V: C4.2, J1.6 (Pin_6), J10.6 (Pin_6), J11.6 (Pin_6), J12.6 (Pin_6), J13.6 (Pin_6), RV3.1, U1.4 (V-), U3.3 (VO), U5.4 (V-)
