File: kicad/led/led.kicad_sch (KiCad schematic)
At the start: 45 parts, among them J1 Conn_01x06, J2 Conn_01x09_Male, U1 LF353DR, U2 LF353DR, U3 LF353DR, U4 LM339DR, U5 LM339DR

Commit message: Maybe finished LED board I think
Parts:
- removed C1, C10, C11, C12, C2, C3, C4, C5, C6, C7, C8, C9: 100n, Capacitor_SMD:C_1206_3216Metric, symbol Device:C
- removed J1: Conn_01x06, Connector_PinHeader_2.54mm:PinHeader_1x06_P2.54mm_Horizontal, symbol Connector_Generic:Conn_01x06
- removed J2: Conn_01x09_Male, Connector_PinHeader_2.54mm:PinHeader_1x09_P2.54mm_Horizontal, symbol Connector:Conn_01x09_Male
- removed RV1, RV3, RV4: 10k, Potentiometer_THT:Potentiometer_Runtron_RM-065_Vertical, symbol Device:R_Potentiometer
- removed U1, U2, U3: LF353DR, Package_SO:SOIC-8_3.9x4.9mm_P1.27mm, symbol Amplifier_Operational:LM358
- removed U4, U5: LM339DR, Package_SO:SO-14_3.9x8.65mm_P1.27mm, symbol Comparator:LM339
- added D1, D13, D17, D21, D25, D29, D33, D37, D5, D9: ORANGE, LED_SMD:LED_1210_3225Metric, symbol Device:LED
- added D10, D14, D18, D2, D22, D26, D30, D34, D38, D6: YELLOW, LED_SMD:LED_1210_3225Metric, symbol Device:LED
- added D11, D15, D19, D23, D27, D3, D31, D35, D39, D7: GREEN, LED_SMD:LED_1210_3225Metric, symbol Device:LED
- added D12, D16, D20, D24, D28, D32, D36, D4, D40, D8: BLUE, LED_SMD:LED_1210_3225Metric, symbol Device:LED
- added J1, J10, J2, J3, J4, J5, J6, J7, J8, J9: Conn_01x04_Male, Connector_PinHeader_2.54mm:PinHeader_1x04_P2.54mm_Horizontal, symbol Connector:Conn_01x04_Male
- added J100: Conn_01x01_Male, Connector_PinSocket_2.54mm:PinSocket_1x01_P2.54mm_Vertical, symbol Connector:Conn_01x01_Male
- added R19, R20, R21, R22, R23, R24, R25, R26, R27, R37, R38, R39, R40, R6, R7, R8, R9: R, Resistor_SMD:R_1206_3216Metric, symbol Device:R
- R1, R2, R3, R4, R5: value 100k -> R
- R10, R11, R12, R28, R29, R30: value 137 -> R
- R13, R14, R15, R31, R32, R33: value 931 -> R
- R16, R17, R18, R34, R35, R36: value 1k87 -> R
Connections:
- net audio_right is gone; now on net +5V: R31.1
- net +5V: now also R1.2, R10.1, R11.1, R12.1, R13.2, R14.1, R15.1, R16.1, R17.2, R18.1, R2.1, R28.1, R29.2, R3.1, R30.1, R32.1, R33.2, R34.1, R35.1, R36.1, R4.1, R5.2, J100.1 (Pin_1), R19.1, R20.1, R21.2, R22.1, R23.1, R24.1, R25.2, R26.1, R27.1, R37.2, R38.1, R39.1, R40.1, R6.1, R7.1, R8.1, R9.2
- net at R31.2: now also D31.2 (A); no longer R28.1
- net at R15.2: now also D15.2 (A); no longer R12.1
- net at R33.1: now also D33.2 (A); no longer R29.2
- net at R17.1: now also D17.2 (A)
- net at R28.2: now also D28.2 (A); no longer R32.1
- net at R30.2: now also D30.2 (A)
- net at R11.2: now also D11.2 (A); no longer R15.1
- net at R2.2: now also D2.2 (A); no longer R3.1
- net at R3.2: now also D3.2 (A); no longer R4.1
- net at R12.2: now also D12.2 (A)
- net at R10.2: now also D10.2 (A); no longer R14.1
- net at R14.2: now also D14.2 (A); no longer R11.1
- net at R4.2: now also D4.2 (A); no longer R5.1
- net at R32.2: now also D32.2 (A); no longer R29.1
- net at R1.1: now also D1.2 (A)
- removed net GND: R16.2, R17.2, R18.2, R34.2, R35.2, R36.2, R5.2
- net audio_left: no longer names the net of R13.1
- net audio_left: now also D13.2 (A)
- new net: D14.1 (K), J4.3 (Pin_3)
- new net: D18.1 (K), J5.3 (Pin_3)
- new net: D18.2 (A), R18.2
- new net: D34.2 (A), R34.2
- new net: D39.2 (A), R39.2
- new net: D37.2 (A), R37.1
- new net: D4.1 (K), J1.1 (Pin_1)
- new net: D36.2 (A), R36.2
- new net: D21.1 (K), J6.1 (Pin_1)
- new net: D22.1 (K), J6.2 (Pin_2)
- new net: D23.1 (K), J6.3 (Pin_3)
- new net: D24.1 (K), J6.4 (Pin_4)
- new net: D11.1 (K), J3.2 (Pin_2)
- new net: D22.2 (A), R22.2
- new net: D23.2 (A), R23.2
- new net: D20.2 (A), R20.2
- new net: D8.1 (K), J2.1 (Pin_1)
- new net: D8.2 (A), R8.2
- new net: D3.1 (K), J1.2 (Pin_2)
- new net: D2.1 (K), J1.3 (Pin_3)
- new net: D1.1 (K), J1.4 (Pin_4)
- new net: D15.1 (K), J4.2 (Pin_2)
- new net: D12.1 (K), J3.1 (Pin_1)
- new net: D10.1 (K), J3.3 (Pin_3)
- new net: D9.1 (K), J3.4 (Pin_4)
- new net: D9.2 (A), R9.1
- new net: D24.2 (A), R24.2
- new net: D5.2 (A), R5.1
- new net: D26.1 (K), J7.2 (Pin_2)
- new net: D26.2 (A), R26.2
- new net: D36.1 (K), J9.4 (Pin_4)
- new net: D39.1 (K), J10.3 (Pin_3)
- new net: D7.1 (K), J2.2 (Pin_2)
- new net: D6.1 (K), J2.3 (Pin_3)
- new net: D5.1 (K), J2.4 (Pin_4)
- new net: D19.1 (K), J5.2 (Pin_2)
- new net: D19.2 (A), R19.2
- new net: D16.1 (K), J4.1 (Pin_1)
- new net: D16.2 (A), R16.2
- new net: D20.1 (K), J5.1 (Pin_1)
- new net: D38.2 (A), R38.2
- new net: D34.1 (K), J9.2 (Pin_2)
- new net: D40.1 (K), J10.4 (Pin_4)
- new net: D40.2 (A), R40.2
- new net: D6.2 (A), R6.2
- new net: D32.1 (K), J8.4 (Pin_4)
- new net: D31.1 (K), J8.3 (Pin_3)
- new net: D17.1 (K), J5.4 (Pin_4)
- new net: D29.1 (K), J8.1 (Pin_1)
- new net: D29.2 (A), R29.1
- new net: D38.1 (K), J10.2 (Pin_2)
- new net: D7.2 (A), R7.2
- new net: D35.1 (K), J9.3 (Pin_3)
- new net: D35.2 (A), R35.2
- new net: D21.2 (A), R21.1
- new net: D37.1 (K), J10.1 (Pin_1)
- new net: D25.2 (A), R25.1
- new net: D25.1 (K), J7.1 (Pin_1)
- new net: D28.1 (K), J7.4 (Pin_4)
- new net: D27.2 (A), R27.2
- new net: D27.1 (K), J7.3 (Pin_3)
- new net: D33.1 (K), J9.1 (Pin_1)
- new net: D13.1 (K), J4.4 (Pin_4)
- new net: D30.1 (K), J8.2 (Pin_2)
Other:
- note removed: "1700 - 5000"
- note removed: "High"
- note removed: "Low"
