File: kicad/power - Copy/power.kicad_pcb (KiCad board)
At the start: 2 copper layers, 22.9 x 17.8 mm, 4 parts, among them J2 AudioJack3, J3 USB_C_Receptacle, U5 LF353DR

Commit message: Made some PCBs
Changed lines of the file:
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@@
     (pad_to_mask_clearance 0)
     (pcbplotparams
-      (layerselection 0x00010fc_ffffffff)
+      (layerselection 0x0001000_7fffffff)
       (disableapertmacros false)
       (usegerberextensions false)
@@
       (outputformat 1)
       (mirror false)
-      (drillshape 1)
+      (drillshape 0)
       (scaleselection 1)
       (outputdirectory "")
@@
   )
   (footprint "audio_footprint:usb_footprint" (layer "F.Cu")
-    (at 203.06 70.68)
+    (at 203.059995 70.679996)
     (property "Sheetfile" "power.kicad_sch")
     (property "Sheetname" "")
@@
       (effects (font (size 1 1) (thickness 0.15)))
     )
-    (pad "A5" smd roundrect (at -0.68 0 90) (size 1.2 0.7) (layers "F.Cu" "F.Paste" "F.Mask") (roundrect_rratio 0.25)
+    (pad "A5" smd roundrect (at -0.82 0 90) (size 1.2 0.7) (layers "F.Cu" "F.Paste" "F.Mask") (roundrect_rratio 0.25)
       (net 3 "unconnected-(J3-PadA5)") (pinfunction "CC1") (pintype "bidirectional"))
-    (pad "A9" smd roundrect (at 1.34 0 90) (size 1.2 0.76) (layers "F.Cu" "F.Paste" "F.Mask") (roundrect_rratio 0.25)
+    (pad "A9" smd roundrect (at 1.2 0 90) (size 1.2 0.76) (layers "F.Cu" "F.Paste" "F.Mask") (roundrect_rratio 0.25)
       (net 2 "+5V") (pinfunction "VBUS") (pintype "passive"))
-    (pad "A12" smd roundrect (at 2.57 0 90) (size 1.2 0.8) (layers "F.Cu" "F.Paste" "F.Mask") (roundrect_rratio 0.25)
+    (pad "A12" smd roundrect (at 2.43 0 90) (size 1.2 0.8) (layers "F.Cu" "F.Paste" "F.Mask") (roundrect_rratio 0.25)
       (net 1 "GND") (pinfunction "GND") (pintype "passive"))
-    (pad "B5" smd roundrect (at 0.32 0 90) (size 1.2 0.7) (layers "F.Cu" "F.Paste" "F.Mask") (roundrect_rratio 0.25)
+    (pad "B5" smd roundrect (at 0.18 0 90) (size 1.2 0.7) (layers "F.Cu" "F.Paste" "F.Mask") (roundrect_rratio 0.25)
       (net 4 "unconnected-(J3-PadB5)") (pinfunction "CC2") (pintype "bidirectional"))
-    (pad "B9" smd roundrect (at -1.7 0 90) (size 1.2 0.76) (layers "F.Cu" "F.Paste" "F.Mask") (roundrect_rratio 0.25)
+    (pad "B9" smd roundrect (at -1.84 0 90) (size 1.2 0.76) (layers "F.Cu" "F.Paste" "F.Mask") (roundrect_rratio 0.25)
       (net 2 "+5V") (pinfunction "VBUS") (pintype "passive"))
-    (pad "B12" smd roundrect (at -2.93 0 90) (size 1.2 0.8) (layers "F.Cu" "F.Paste" "F.Mask") (roundrect_rratio 0.25)
+    (pad "B12" smd roundrect (at -3.07 0 90) (size 1.2 0.8) (layers "F.Cu" "F.Paste" "F.Mask") (roundrect_rratio 0.25)
       (net 1 "GND") (pinfunction "GND") (pintype "passive"))
-    (pad "S1" thru_hole oval (at -4.64 0 90) (size 1.7 1.1) (drill oval 1.2 0.6) (layers *.Cu *.Mask)
+    (pad "S1" thru_hole circle (at 4 3.8 90) (size 1.7 1.7) (drill 1.2) (layers *.Cu *.Mask)
       (net 1 "GND") (pinfunction "SHIELD") (pintype "passive"))
-    (pad "S1" thru_hole oval (at 4 3.8 90) (size 1.7 1.1) (drill oval 1.2 0.6) (layers *.Cu *.Mask)
+    (pad "S1" thru_hole circle (at -4.64 0 90) (size 1.7 1.7) (drill 1.2) (layers *.Cu *.Mask)
       (net 1 "GND") (pinfunction "SHIELD") (pintype "passive"))
-    (pad "S1" thru_hole oval (at 4 0 90) (size 1.7 1.1) (drill oval 1.2 0.6) (layers *.Cu *.Mask)
+    (pad "S1" thru_hole circle (at 4 0 90) (size 1.7 1.7) (drill 1.2) (layers *.Cu *.Mask)
       (net 1 "GND") (pinfunction "SHIELD") (pintype "passive"))
-    (pad "S1" thru_hole oval (at -4.64 3.8 90) (size 1.7 1.1) (drill oval 1.2 0.6) (layers *.Cu *.Mask)
+    (pad "S1" thru_hole circle (at -4.64 3.8 90) (size 1.7 1.7) (drill 1.2) (layers *.Cu *.Mask)
       (net 1 "GND") (pinfunction "SHIELD") (pintype "passive"))
+    (group "" (id 062fbe79-da43-4e6a-bd6f-509557f2df9b)
+      (members
+        2b894b8a-c098-4d9d-be0f-2ef41dea274e
+        5f74c6fb-337b-40a9-9b79-933f2f30429a
+        a9ad6ea5-8293-424c-89d4-c01baf033429
+        d36e7ed4-f2bc-4d88-86ae-317d3c24af1a
+        dbd87a35-3166-440e-a8f0-c71d214a12a6
+        ff203a9b-3d2e-4e1d-a6f0-12d16e5120fb
+      )
+    )
+    (group "" (id 7147b342-4ca8-4694-a1ec-b615c151a5d0)
+      (members
+        3ce4c631-4e8b-4ee6-a520-34bf7b12880c
+        4116bfc2-eab3-4c29-a983-44eacd9f10f5
+        51320c8c-9c4a-48b8-a7b8-e2c8d1f2e5ad
+        704ba6e6-ee13-4d9d-b544-d836a743bdda
+      )
+    )
   )
   (footprint "audio_footprint:audio_jack" (layer "F.Cu")
