File: kicad/filter/filter.kicad_pcb (KiCad board)
At the start: 2 copper layers, 73 x 25.1 mm, 45 parts, among them J1 Conn_01x06, J2 Conn_01x09_Male, U1 LF353DR, U2 LF353DR, U3 LF353DR, U4 LM339DR, U5 LM339DR

Commit message: Made some PCBs
Routing:
- net -15V: track 46.4 -> 41.5 mm
Changed lines of the file:
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@@
   (segment (start 145.415 73.279) (end 145.542 73.406) (width 0.635) (layer "F.Cu") (net 5))
   (segment (start 126.619 73.406) (end 121.158 67.945) (width 0.635) (layer "F.Cu") (net 5))
-  (segment (start 121.158 67.945) (end 122.682 69.469) (width 0.635) (layer "B.Cu") (net 5))
-  (segment (start 122.682 69.469) (end 122.682 70.866) (width 0.635) (layer "B.Cu") (net 5))
-  (segment (start 122.682 70.866) (end 123.571 71.755) (width 0.635) (layer "B.Cu") (net 5))
   (segment (start 149.225 76.77) (end 149.225 75.184) (width 0.635) (layer "F.Cu") (net 6))
   (segment (start 137.922 75.184) (end 123.317 75.184) (width 0.635) (layer "F.Cu") (net 6))

Commit message: Preparing to maybe do V2 of power
Parts:
- C1: renamed from R10; value 137 -> 93.1
- C10: renamed from C6; value 100n -> DNP
- C11: renamed from R18; value 1k87 -> 330
- C12: renamed from R28; value 137 -> 93.1
- C13: renamed from R29; value 137 -> 226
- C14: renamed from R30; value 137 -> 307
- C15: renamed from R31; value 931 -> 100n
- C16: renamed from R32; value 931 -> 100n
- C17: renamed from R33; value 931 -> 100n
- C18: renamed from C10; value 100n -> DNP
- C19: renamed from R34; value 1k87 -> 1k10
- C2: renamed from R11; value 137 -> 226
- C20: renamed from C11; value 100n -> DNP
- C21: renamed from R35; value 1k87 -> 453
- C22: renamed from C12; value 100n -> DNP
- C23: renamed from R36; value 1k87 -> 330
- C3: renamed from R12; value 137 -> 307
- C4: renamed from R13; value 931 -> 100n
- C5: renamed from R14; value 931 -> 100n
- C6: renamed from R15; value 931 -> 100n
- C7: renamed from R16; value 1k87 -> 1k10
- C8: renamed from C5; value 100n -> DNP
- C9: renamed from R17; value 1k87 -> 453
- Z1: renamed from C4; value 100n -> DNP
- renumbered C8 to R10, C9 to R11, C1 to R6, C2 to R7, C3 to R8, C7 to R9
